File: paw3222-pcb/PAW3222.kicad_sch (KiCad schematic)
At the start: 7 parts, among them J1 Conn_01x06_Socket, U1 PAW3220LU

Commit message: add led
Parts:
- removed R2: 10kΩ, Resistor_SMD:R_0603_1608Metric, symbol Device:R
- added D1: IR LED LTE-C216-P-W, paw3222:LTE-C216-P-W, symbol Device:LED
- C1, C2, C3: footprint Capacitor_SMD:C_0603_1608Metric -> Capacitor_SMD:C_0402_1005Metric
- R1: value 10kΩ -> 51R; footprint Resistor_SMD:R_0603_1608Metric -> Resistor_SMD:R_0402_1005Metric
Connections:
- net MOTION: no longer R1.1
- net at U1.E1 (LED): now also D1.1 (K)
- new net: D1.2 (A), R1.1
Other:
- moved on the sheet: C3

Commit message: delete r
Parts:
- removed R1: 51R, Resistor_SMD:R_0402_1005Metric, symbol Device:R
Connections:
- net VCC 3.3V: now also D1.2 (A)
Changed lines of the file:
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@@
-	(wire
-		(pts
-			(xy 135.89 102.87) (xy 139.7 102.87)
-		)
-		(stroke
-			(width 0)
-			(type default)
-		)
-	)
 	(wire
 		(pts
@@
 	(wire
 		(pts
-			(xy 121.92 102.87) (xy 128.27 102.87)
+			(xy 121.92 102.87) (xy 139.7 102.87)
 		)
 		(stroke
@@
 					(unit 1)
 				)
-			)
-		)
-	)
-	(symbol
-		(lib_id "Device:R")
-		(at 132.08 102.87 90)
-		(unit 1)
-		(exclude_from_sim no)
-		(in_bom yes)
-		(on_board yes)
-		(dnp no)
-		(property "Reference" "R1"
-			(at 132.08 97.79 90)
-			(effects
-				(font
-					(size 1.27 1.27)
-				)
-			)
-		)
-		(property "Value" "51R"
-			(at 132.08 100.33 90)
-			(effects
-				(font
-					(size 1.27 1.27)
-				)
-			)
-		)
-		(property "Footprint" "Resistor_SMD:R_0402_1005Metric"
-			(at 132.08 104.648 90)
-			(effects
-				(font
-					(size 1.27 1.27)
-				)
-				(hide yes)
-			)
-		)
-		(property "Datasheet" "~"
-			(at 132.08 102.87 0)
-			(effects
-				(font
-					(size 1.27 1.27)
-				)
-				(hide yes)
-			)
-		)
-		(property "Description" "Resistor"
-			(at 132.08 102.87 0)
-			(effects
-				(font
-					(size 1.27 1.27)
-				)
-				(hide yes)
-			)
-		)
-		(property "LCSC" ""
-			(at 132.08 102.87 90)
-			(effects
-				(font
-					(size 1.27 1.27)
-				)
-				(hide yes)
-			)
-		)
-		(pin "1"
-		)
-		(pin "2"
-		)
-		(instances
-			(project "PAW3222"
-				(path "/09dfddcd-8b98-44c2-a619-d4f9ad8a2432"
-					(reference "R1")
-					(unit 1)
-				)
