File: paw3222-pcb/PAW3222.kicad_pcb (KiCad board)
At the start: 2 copper layers, 11 x 13 mm, 7 parts, among them J1 Conn_01x06_Socket, U1 PAW3220LU

Commit message: add led
Parts:
- removed R2: 10kΩ, Resistor_SMD:R_0603_1608Metric
- added D1: IR LED LTE-C216-P-W, paw3222:LTE-C216-P-W, F.Cu at (143.1, 85.8)
- C1, C2, C3: footprint Capacitor_SMD:C_0603_1608Metric -> Capacitor_SMD:C_0402_1005Metric
- R1: value 10kΩ -> 51R; footprint Resistor_SMD:R_0603_1608Metric -> Resistor_SMD:R_0402_1005Metric
- moved C1 3.03 mm to (147.5, 82.0)
- moved C2 1.78 mm to (147.5, 80.0)
- moved C3 0.51 mm to (147.5, 78.0)
Connections:
- R1 pad 1: MOTION -> Net-(D1-A)
- U1 pad E1: unconnected-(U1-LED-PadE1) -> Net-(D1-K)
Routing:
- net Net-(D1-A): track 0.00 -> 14.8 mm
- net SDIO: track 20.3 -> 9.48 mm, vias 3 -> 2
- net VCC 3.3V: track 32.9 -> 22.1 mm, vias 2 -> 0
- net MOTION: track 12.7 -> 3.27 mm, vias 2 -> 0
- net Net-(D1-K): track 0.00 -> 5.44 mm
- net Net-(U1-VDDA): track 7.90 -> 8.53 mm

Commit message: delete r
Parts:
- removed R1: 51R, Resistor_SMD:R_0402_1005Metric
- moved C3 8.31 mm to (139.2, 79.0)
- moved C1 2.51 mm to (147.2, 79.5), turned to 0 degrees
- moved C2 1.52 mm to (147.2, 78.5), turned to 0 degrees
Connections:
- D1 pad 2: Net-(D1-A) -> VCC 3.3V
Routing:
- net Net-(D1-A): track 14.8 -> 0.00 mm
- net VCC 3.3V: track 22.1 -> 13.9 mm
- net GND: track 22.3 -> 18.0 mm
- net Net-(U1-VDDA): track 8.53 -> 6.24 mm
- net Net-(D1-K): track 5.44 -> 3.94 mm
- net SDIO: track 9.48 -> 8.62 mm

Commit message: 基板修正
Routing:
- net GND: track 18.0 -> 17.0 mm
Changed lines of the file:
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@@
 		)
 		(fp_text user "+"
-			(at 0.82 1.81 90)
+			(at -0.65 3.15 90)
 			(unlocked yes)
 			(layer "Dwgs.User")
@@
 		(fp_circle
 			(center -2.7 5.425)
-			(end -2 5.425)
-			(stroke
-				(width 0.1)
-				(type default)
+			(end -1.8 5.425)
+			(stroke
+				(width 0.1)
+				(type solid)
 			)
 			(fill no)
@@
 		(pad "A1" smd circle
 			(at -0.44 -0.6)
-			(size 0.25 0.25)
+			(size 0.3 0.3)
 			(layers "F.Cu" "F.Mask" "F.Paste")
 			(net 2 "Net-(U1-VDDA)")
@@
 		(pad "A3" smd circle
 			(at 0.44 -0.6)
-			(size 0.25 0.25)
+			(size 0.3 0.3)
 			(layers "F.Cu" "F.Mask" "F.Paste")
 			(net 5 "NCS")
@@
 		(pad "B2" smd circle
 			(at 0 -0.3)
-			(size 0.25 0.25)
+			(size 0.3 0.3)
 			(layers "F.Cu" "F.Mask" "F.Paste")
 			(net 6 "MOTION")
@@
 		(pad "C1" smd circle
 			(at -0.44 0)
-			(size 0.25 0.25)
+			(size 0.3 0.3)
 			(layers "F.Cu" "F.Mask" "F.Paste")
 			(net 1 "GND")
@@
 		(pad "C3" smd circle
 			(at 0.44 0)
-			(size 0.25 0.25)
+			(size 0.3 0.3)
 			(layers "F.Cu" "F.Mask" "F.Paste")
 			(net 3 "SDIO")
@@
 		(pad "D2" smd circle
 			(at 0 0.3)
-			(size 0.25 0.25)
+			(size 0.3 0.3)
 			(layers "F.Cu" "F.Mask" "F.Paste")
 			(net 7 "SCLK")
@@
 		(pad "E1" smd circle
 			(at -0.44 0.6)
-			(size 0.25 0.25)
+			(size 0.3 0.3)
 			(layers "F.Cu" "F.Mask" "F.Paste")
 			(net 8 "Net-(D1-K)")
@@
 		(pad "E3" smd circle
 			(at 0.44 0.6)
-			(size 0.25 0.25)
+			(size 0.3 0.3)
 			(layers "F.Cu" "F.Mask" "F.Paste")
 			(net 4 "VCC 3.3V")
@@
 	)
 	(segment
+		(start 147 77.5)
+		(end 147.75 78.25)
+		(width 0.25)
+		(layer "F.Cu")
+		(net 1)
+	)
+	(segment
 		(start 141.4 82.6)
 		(end 141.6 82.8)
@@
 	)
 	(segment
+		(start 141.75 78.5)
+		(end 141.75 79.5)
+		(width 0.25)
+		(layer "F.Cu")
+		(net 1)
+	)
+	(segment
 		(start 141.6 82.8)
 		(end 142.57 82.8)
@@
 	)
 	(segment
-		(start 141.75 77.5)
-		(end 141.75 79.5)
+		(start 142.75 77.5)
+		(end 141.75 78.5)
 		(width 0.25)
 		(layer "F.Cu")
@@
 	)
 	(segment
-		(start 147.75 77.5)
+		(start 147.75 78.48)
+		(end 147.73 78.5)
+		(width 0.25)
+		(layer "F.Cu")
+		(net 1)
+	)
+	(segment
+		(start 147.75 78.25)
 		(end 147.75 78.48)
 		(width 0.25)
@@
 	)
 	(segment
-		(start 147.75 78.48)
-		(end 147.73 78.5)
-		(width 0.25)
-		(layer "F.Cu")
-		(net 1)
-	)
-	(segment
 		(start 147.73 78.5)
 		(end 147.73 79.5)
@@
 	)
 	(via
-		(at 141.75 77.5)
+		(at 142.75 77.5)
 		(size 0.45)
 		(drill 0.3)
@@
 	)
 	(via
-		(at 147.75 77.5)
+		(at 147 77.5)
 		(size 0.45)
 		(drill 0.3)
@@
 	)
 	(segment
-		(start 146.75 77.5)
-		(end 141.75 77.5)
-		(width 0.25)
-		(layer "B.Cu")
-		(net 1)
-	)
-	(segment
-		(start 146.75 77.5)
-		(end 147.75 77.5)
+		(start 142.75 77.5)
+		(end 147 77.5)
 		(width 0.25)
 		(layer "B.Cu")
@@
 	)
 	(segment
+		(start 143.06 81.94)
+		(end 143.06 82.55)
+		(width 0.16)
+		(layer "F.Cu")
+		(net 6)
+	)
+	(segment
 		(start 143.25 81.75)
 		(end 143.06 81.94)
 		(width 0.16)
 		(layer "F.Cu")
-		(net 6)
-	)
-	(segment
-		(start 143.06 81.94)
-		(end 143.06 82.55)
-		(width 0.16)
-		(layer "F.Cu")
-		(net 6)
-	)
-	(arc
-		(start 143.1 82.51)
-		(mid 143.088284 82.538284)
-		(end 143.06 82.55)
-		(width 0.16)
-		(layer "F.Cu")

Commit message: pcb最新化
Parts:
- moved J1 1.49 mm to (143.0, 69.8)
Routing:
- net NCS: track 2.98 -> 4.43 mm
- net MOTION: track 3.21 -> 4.62 mm
- net VCC 3.3V: track 13.9 -> 12.5 mm
- net SDIO: track 8.62 -> 7.38 mm
- net SCLK: track 6.48 -> 7.53 mm
- net Net-(D1-K): track 3.94 -> 3.11 mm
- net GND: track 17.0 -> 16.7 mm, vias 2 -> 12
Other:
- board size 11 x 13 mm -> 11 x 14.5 mm
